File: RF_Remote.kicad_pcb (KiCad board)
At the start: 2 copper layers, 90 parts, among them J1 JTAG, J2 UART, J6 CH_USB_C, SW1 NRST, SW2 BOOT, SW3 NRST, SW4 NRST, U2 AP7343D-33W5, U3 MICRF112YMU-TR, U4 MCP73833, Y1 25MHz, Y2 32.786KHz, Y3 13.56MHz

Commit message: Routing progress
Parts:
- removed the TP2 at (95.8, 122.7)
- added TP6: 3v3, TestPoint:TestPoint_Pad_D1.5mm, F.Cu at (100.4, 118.5)
- added TP7: GND, TestPoint:TestPoint_Pad_D1.5mm, F.Cu at (102.9, 118.5)
- added U5: STM32U031G6Yx, Package_CSP:ST_WLCSP-27_2.34x2.55mm_Layout9x6_P0.4mm_Stagger, F.Cu at (98.3, 99.4)
- moved J2 75.2 mm to (80.1, 128.2)
- moved U2 67.7 mm to (97.4, 118.1)
- moved R17 55.5 mm to (106.1, 132.5), turned to 90 degrees
- moved C22 49.9 mm to (97.3, 123.7), turned to 180 degrees
- moved R18 46.4 mm to (103.8, 125.8), turned to 180 degrees
- moved R19 45.6 mm to (103.8, 127.3), turned to 180 degrees
- moved R20 44.8 mm to (103.8, 128.8), turned to 180 degrees
- moved D12 40.0 mm to (100.7, 125.8), turned to 180 degrees
- moved D13 39.4 mm to (100.7, 127.3), turned to 180 degrees
- moved C15 39.1 mm to (98.1, 121.4), turned to 90 degrees
- moved D14 38.9 mm to (100.7, 128.8), turned to 180 degrees
- moved C18 37.3 mm to (94.3, 117.5)
- moved U4 37.2 mm to (100.7, 122.3), turned to 90 degrees
- moved C27 36.8 mm to (96.6, 121.4), turned to -90 degrees
- moved R21 36.8 mm to (103.2, 121.7), turned to 90 degrees
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- renumbered C12 to C10, C13 to C12, C14 to C13, C15 to C14, C16 to C15, C17 to C16, C18 to C17, C19 to C18, C20 to C19, C21 to C20, C22 to C21, C23 to C22, C24 to C23, C25 to C24, C26 to C25, C27 to C26, C28 to C27, C4 to C3, C3 to C4, C6 to C5, C5 to C6, C9 to C8, C10 to C9, D11 to D1, D3 to D11, D4 to D12, D5 to D13, D6 to D14, D1 to D2, D12 to D3, D2 to D4, D13 to D5, D14 to D6, J6 to J3, R22 to R10, R5 to R11, R15 to R12, R16 to R13, R6 to R14, R17 to R15, R18 to R16, R7 to R17, R9 to R18, R10 to R19, R11 to R20, R12 to R21, R19 to R3, R3 to R4, R20 to R5, R13 to R6, R14 to R7, R4 to R8, R21 to R9, TP3 to TP1, TP4 to TP2, TP1 to TP3, TP5 to TP4, TP6 to TP5
Connections:
- J1 pad 6: /SWO -> unconnected-(J1-SWO-Pad6)
Routing:
- net Net-(U4-~{PG}): track 0.00 -> 13.3 mm
- net Net-(U4-STAT2): track 0.00 -> 7.47 mm
- net Net-(J3-CC1): track 4.75 -> 10.6 mm
- net Net-(U4-STAT1): track 0.00 -> 5.32 mm
- net GND: track 4.04 -> 8.56 mm, vias 2 -> 5
- net Net-(U4-THERM): track 0.00 -> 4.41 mm, vias 0 -> 1
- net Net-(F1-Pad1): track 9.48 -> 6.76 mm
- net Net-(D14-K): track 0.00 -> 1.44 mm
- net Net-(D13-K): track 0.00 -> 1.44 mm
- net Net-(D12-K): track 0.00 -> 1.44 mm
- added copper zone on F.Cu, net GND
- added copper zone on F.Cu, net Net-(D11-K)
- added copper zone on F.Cu, net Net-(F1-Pad1)
- added copper zone on F.Cu, net Net-(U4-PROG)

Commit message: Layout progress
Parts:
- removed the C10 at (129.8, 88.5)
- removed the C13 at (129.8, 93.5)
- removed the C17 at (129.8, 103.5)
- removed C23: 1p2, Capacitor_SMD:C_0603_1608Metric
- removed C24: 2p2, Capacitor_SMD:C_0603_1608Metric
- removed C25: dnp, Capacitor_SMD:C_0603_1608Metric
- removed C26: 6p8, Capacitor_SMD:C_0603_1608Metric
- removed the C8 at (125.8, 103.5)
- removed the C8 at (125.8, 106.0)
- removed the TP4 at (161.8, 105.5)
- removed the TP5 at (161.8, 109.0)
- removed U5: STM32U031G6Yx, Package_CSP:ST_WLCSP-27_2.34x2.55mm_Layout9x6_P0.4mm_Stagger
- removed Y3: 13.56MHz, Crystal:Crystal_SMD_3225-4Pin_3.2x2.5mm
- added C15: 12p, Capacitor_SMD:C_0603_1608Metric, F.Cu at (127.6, 49.1)
- added C18: 1p2, Capacitor_SMD:C_0603_1608Metric, F.Cu at (131.6, 36.5)
- added C8: 100n, Capacitor_SMD:C_0603_1608Metric, B.Cu at (103.2, 116.7)
- added JP3: A/F-SK, Jumper:SolderJumper-3_P2.0mm_Open_TrianglePad1.0x1.5mm_NumberLabels, F.Cu at (132.9, 50.9)
- added U1: STM32U031G6Yx, Package_CSP:ST_WLCSP-27_2.34x2.55mm_Layout9x6_P0.4mm_Stagger, F.Cu at (101.5, 117.6)
- BT1, C1, C5, D11, D12, D13, D14, F1, J3, JP1, L1, R17, R18, R19, R20, R21, SW1, SW2, U2, U4: moved to B.Cu
- C10: renamed from C15; moved to B.Cu
- C12: value 100n -> 10u
- C13: renamed from C18; moved to B.Cu
- C14: value 100p -> 12p
- C16: value 100n -> dnp
- C17: renamed from C22; moved to B.Cu
- C19: value 12p -> 2p2
- C2: value 4u7 -> 100n
- C20: value 12p -> dnp
- C21: value dnp -> 6p8
- C22: renamed from C27; moved to B.Cu
- C4: value 100n -> 4u7; moved to B.Cu
- C7: value 100n -> 12p
- C9: value 100n -> 100p
- D10: value 0 -> STATUS
- D2: value PWR -> 2
- D3: value 2 -> 1
- D4: value STATUS -> 0
- D5: value 1 -> 3
- D6: value 0 -> 2
- D7: value 3 -> 1
- D8: value 2 -> 0
- D9: value 1 -> PWR; moved to B.Cu
- JP2: value A/F-SK -> SENS; footprint Jumper:SolderJumper-3_P2.0mm_Open_TrianglePad1.0x1.5mm_NumberLabels -> Jumper:SolderJumper-2_P1.3mm_Open_TrianglePad1.0x1.5mm; moved to B.Cu
- R1, R2: value 10k -> 1k
- R10, R8: value 1k -> 10k; moved to B.Cu
- R11: value 10k -> 5k1; moved to B.Cu
- R13: value 1k -> 20k; moved to B.Cu
- R14: value 10k -> 30k; moved to B.Cu
- R15, R16: value 1k -> 10k
- R4: value 5k1 -> 1k
- R6: value 20k -> 1k
- R7: value 30k -> 1k
- TP2: value RX -> TX
- TP3: value TX -> RX
- TP4: renamed from TP6; moved to B.Cu
- TP5: renamed from TP7; moved to B.Cu
- Y1: value 25MHz -> 32.786KHz; footprint Crystal:Crystal_SMD_3225-4Pin_3.2x2.5mm -> Crystal:Crystal_SMD_3215-2Pin_3.2x1.5mm
- Y2: value 32.786KHz -> 13.56MHz; footprint Crystal:Crystal_SMD_3215-2Pin_3.2x1.5mm -> Crystal:Crystal_SMD_3225-4Pin_3.2x2.5mm
- moved J1 132.1 mm to (47.1, 24.0)
- moved TP1 110.2 mm to (70.0, 39.4)
- moved TP2 110.2 mm to (70.0, 43.0)
- moved TP3 103.2 mm to (70.0, 46.5)
- moved SW1 86.4 mm to (75.3, 134.9), turned to 180 degrees
- moved R7 83.6 mm to (59.9, 102.7), turned to -90 degrees
- moved R9 83.5 mm to (58.4, 102.7), turned to -90 degrees
- moved J2 81.8 mm to (74.7, 46.6), turned to 180 degrees
- moved SW2 78.9 mm to (81.2, 134.9), turned to 180 degrees
- moved Y2 78.8 mm to (121.7, 48.1)
- moved R5 78.8 mm to (63.0, 102.7), turned to -90 degrees
- moved R6 76.6 mm to (61.5, 102.7), turned to -90 degrees
- moved R3 75.8 mm to (66.1, 102.7), turned to -90 degrees
- moved R12 75.8 mm to (66.2, 91.9)
- moved R4 75.2 mm to (64.6, 102.7), turned to -90 degrees
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Connections:
- C11 pad 1: GND -> +3V3
- C11 pad 2: /WKUP_2 -> GND
- C12 pad 1: +3.3VA -> +3V3
- C14 pad 1: +3V3 -> GND
- C14 pad 2: GND -> Net-(U3-XTLIN)
- C16 pad 1: +3V3 -> Net-(U3-XTAL_MOD)
- C16 pad 2: GND -> Net-(U3-XTLOUT)
- C19 pad 1: GND -> Net-(U3-PAOUT)
- C19 pad 2: Net-(U3-XTLIN) -> Net-(C19-Pad2)
- C2 pad 1: +3V3 -> GND
- C2 pad 2: GND -> /WKUP_1
- C20 pad 1: GND -> Net-(C19-Pad2)
- C20 pad 2: Net-(U3-XTLOUT) -> GND
- C21 pad 1: Net-(U3-XTAL_MOD) -> Net-(AE1-A)
- C21 pad 2: Net-(U3-XTLOUT) -> GND
- C3 pad 2: /HSE_I -> /LSE_I
- C5 pad 1: GND -> +3V3
- C5 pad 2: /WKUP_1 -> GND
- C6 pad 1: +3V3 -> GND
- C6 pad 2: GND -> /WKUP_2
- C7 pad 1: +3V3 -> GND
- C7 pad 2: GND -> /LSE_O
- D10 pad 1: /DATA0 -> /STATUS
- D2 pad 1: GND -> /DATA6
- D3 pad 1: /DATA6 -> /DATA5
- D4 pad 1: /STATUS -> /DATA4
- D5 pad 1: /DATA5 -> /DATA3
- D6 pad 1: /DATA4 -> /DATA2
- D7 pad 1: /DATA3 -> /DATA1
- D8 pad 1: /DATA2 -> /DATA0
- D9 pad 1: /DATA1 -> GND
- JP2 pad 2: /RF_TX -> +BATT
- L3 pad 1: Net-(C24-Pad2) -> Net-(C19-Pad2)
- R1 pad 1: /NRST -> Net-(D1-A)
- R10 pad 1: Net-(D6-A) -> GND
- R10 pad 2: +3V3 -> /BOOT
- R11 pad 1: /WKUP_1 -> Net-(D9-A)
- R11 pad 2: +3V3 -> Net-(JP1-A)
- R12 pad 1: Net-(D7-A) -> Net-(D10-A)
- R13 pad 1: Net-(D8-A) -> Net-(JP2-A)
- R13 pad 2: +3V3 -> Net-(U1-PA4)
- R14 pad 1: /WKUP_2 -> Net-(U1-PA4)
- R14 pad 2: +3V3 -> GND
- R15 pad 1: Net-(D9-A) -> /WKUP_1
- R16 pad 1: Net-(D10-A) -> /WKUP_2
- R2 pad 1: GND -> Net-(D2-A)
- R2 pad 2: /BOOT -> +3V3
- R3 pad 1: Net-(D1-A) -> Net-(D3-A)
- R4 pad 1: Net-(D2-A) -> Net-(D4-A)
- R4 pad 2: Net-(JP1-A) -> +3V3
- R5 pad 1: Net-(D3-A) -> Net-(D5-A)
- R6 pad 1: +BATT -> Net-(D6-A)
- R6 pad 2: Net-(U5-PA4) -> +3V3
- R7 pad 1: Net-(U5-PA4) -> Net-(D7-A)
- R7 pad 2: GND -> +3V3
- R8 pad 1: Net-(D4-A) -> /NRST
- R9 pad 1: Net-(D5-A) -> Net-(D8-A)
- TP1 pad 1: Net-(J2-Pin_3) -> /RF_TX
- TP2 pad 1: Net-(J2-Pin_2) -> Net-(J2-Pin_3)
- TP3 pad 1: /RF_TX -> Net-(J2-Pin_2)
- U3 pad 1: Net-(JP2-B) -> Net-(JP3-B)
- U3 pad 6: Net-(JP2-A) -> Net-(JP3-A)
- Y1 pad 1: /HSE_I -> /LSE_I
- Y1 pad 2: GND -> /LSE_O
- Y2 pad 1: /LSE_I -> Net-(U3-XTLIN)
- Y2 pad 2: /LSE_O -> GND
Routing:
- net +3V3: track 0.00 -> 15.8 mm, vias 0 -> 12
- net Net-(U1-PA4): track 0.00 -> 9.37 mm, vias 0 -> 2
- net /DATA6: track 0.00 -> 8.60 mm, vias 0 -> 2
- net /DATA0: track 0.00 -> 7.03 mm
- net GND: track 8.56 -> 15.1 mm, vias 5 -> 19
- net /LSE_I: track 0.00 -> 6.22 mm
- net /DATA1: track 0.00 -> 5.93 mm
- net +BATT: track 0.00 -> 5.70 mm
- net /DATA7: track 0.00 -> 5.55 mm
- net /RF_EN: track 0.00 -> 5.32 mm
- net /LSE_O: track 0.00 -> 5.21 mm
- net /RF_TX: track 0.00 -> 4.81 mm
- net +3.3VA: track 0.00 -> 4.14 mm, vias 0 -> 1
- net /DATA2: track 0.00 -> 3.53 mm, vias 0 -> 1
- net Net-(U4-THERM): track 4.41 -> 0.88 mm
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- added copper zone on B.Cu, net +3V3
- added copper zone on In2.Cu, net +3V3
- added copper zone on B.Cu, net +BATT
- added copper zone on B.Cu, net GND
- added copper zone on In1.Cu, net GND
- added copper zone on B.Cu, net Net-(D11-K)
- added copper zone on B.Cu, net Net-(F1-Pad1)
- added copper zone on B.Cu, net Net-(U4-PROG)
- removed copper zone on F.Cu, net Net-(D11-K)
- removed copper zone on F.Cu, net Net-(F1-Pad1)
- removed copper zone on F.Cu, net Net-(U4-PROG)
Other:
- board outline added: 25 x 42.5 mm
- copper layers 2 -> 4
- board text added: "PWR"

Commit message: Layout v1
Parts:
- removed TP1: TX, TestPoint:TestPoint_Pad_D1.5mm
- removed the TP2 at (70.0, 43.0)
- removed the TP3 at (70.0, 46.5)
- added AE1: Antenna, TestPoint:TestPoint_THTPad_D1.0mm_Drill0.5mm, B.Cu at (94.7, 87.4)
- C11, C12, C14, C15, C16, C18, C19, C20, C21, C9, JP3, L2, L3, U3, Y2: moved to B.Cu
- moved J1 94.0 mm to (107.2, 96.3)
- moved J2 78.1 mm to (93.8, 122.3)
- moved C16 75.4 mm to (105.9, 104.9)
- moved C18 74.8 mm to (95.1, 101.8), turned to -135 degrees
- moved C19 68.5 mm to (94.7, 96.8), turned to 90 degrees
- moved U3 67.9 mm to (99.7, 102.3), turned to 180 degrees
- moved C9 66.9 mm to (98.4, 99.2), turned to 90 degrees
- moved C20 64.9 mm to (94.0, 94.5), turned to 180 degrees
- moved C11 64.0 mm to (99.9, 99.2), turned to 90 degrees
- moved JP3 63.7 mm to (99.7, 105.2)
- moved L2 62.9 mm to (95.8, 99.2)
- moved C12 61.0 mm to (101.5, 99.2), turned to 90 degrees
- moved C14 61.0 mm to (102.9, 102.3), turned to 90 degrees
- moved C21 58.9 mm to (94.0, 89.3), turned to 180 degrees
- moved Y2 56.5 mm to (105.9, 102.3)
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- renumbered TP4 to TP2, TP5 to TP3
Routing:
- net GND: track 15.1 -> 62.0 mm, vias 19 -> 26
- net +3V3: track 15.8 -> 26.6 mm, vias 12 -> 14
- net Net-(U3-XTLOUT): track 0.00 -> 10.1 mm
- net /WKUP_1: track 1.36 -> 10.9 mm
- net /WKUP_2: track 1.15 -> 10.6 mm
- net /NRST: track 3.02 -> 10.6 mm
- net Net-(U3-PAOUT): track 0.00 -> 7.07 mm
- net /BOOT: track 1.98 -> 7.83 mm
- net Net-(JP3-B): track 0.00 -> 5.49 mm, vias 0 -> 2
- net Net-(U3-XTAL_MOD): track 0.00 -> 4.79 mm
- net Net-(U3-XTLIN): track 0.00 -> 3.97 mm
- net Net-(AE1-A): track 0.00 -> 3.40 mm
- net Net-(C19-Pad2): track 0.00 -> 3.05 mm
- net Net-(JP3-A): track 0.00 -> 2.18 mm
- added copper zone on In1.Cu, net +3V3
- added copper zone on In2.Cu, net GND
- removed copper zone on In2.Cu, net +3V3
- removed copper zone on In1.Cu, net GND
Other:
- board size 25 x 42.5 mm -> 19 x 55 mm
- board text added: "BOOT"
- board text added: "BTN0"
- board text added: "BTN1"
- board text added: "DATA"
- board text added: "NRST"
- board text added: "STATUS"

Commit message: Cleaned up layout
Parts:
- removed the J2 at (93.8, 122.3)
- added C5: 100n, Capacitor_SMD:C_0603_1608Metric, F.Cu at (98.7, 108.9)
- C3: renamed from C4; moved to F.Cu
- C6: renamed from C5; moved to F.Cu
- TH1: moved to B.Cu
- U1: value STM32U031G6Yx -> STM32U031K4Ux; footprint Package_CSP:ST_WLCSP-27_2.34x2.55mm_Layout9x6_P0.4mm_Stagger -> Package_DFN_QFN:QFN-32-1EP_5x5mm_P0.5mm_EP3.45x3.45mm
- moved C3 7.90 mm to (98.7, 107.4), turned to 0 degrees
- moved TH1 7.31 mm to (94.2, 121.4), turned to -90 degrees
- moved C8 6.35 mm to (95.6, 114.6), turned to 180 degrees
- moved C9 6.02 mm to (98.8, 112.6)
- moved C6 5.40 mm to (105.5, 115.7), turned to -90 degrees
- moved Y1 5.24 mm to (95.6, 111.8), turned to 90 degrees
- moved C4 4.61 mm to (95.6, 108.9), turned to 180 degrees
- moved U1 4.50 mm to (101.5, 113.1), turned to 0 degrees
- moved L1 4.49 mm to (99.0, 114.2), turned to 180 degrees
- moved J1 0.49 mm to (106.8, 96.2), turned to 180 degrees
- renumbered C9 to C10, C10 to C11, C11 to C12, C12 to C13, C13 to C14, C14 to C15, C15 to C16, C16 to C17, C17 to C18, C18 to C19, C19 to C20, C20 to C21, C21 to C22, C22 to C23, C3 to C4, C6 to C7, C7 to C8, C8 to C9, J3 to J2, TP2 to TP1, TP3 to TP2
Connections:
- J1 pad 6: unconnected-(J1-SWO-Pad6) -> /SWO
Routing:
- net /STATUS: track 1.60 -> 32.8 mm, vias 1 -> 2
- net /NRST: track 10.6 -> 41.4 mm, vias 0 -> 2
- net /WKUP_2: track 10.6 -> 36.1 mm, vias 1 -> 2
- net /DATA4: track 3.23 -> 27.7 mm, vias 0 -> 2
- net /DATA3: track 3.43 -> 26.0 mm, vias 0 -> 2
- net /SWO: track 0.00 -> 21.0 mm
- net /DATA2: track 3.53 -> 24.2 mm, vias 1 -> 2
- net /SWDIO: track 0.00 -> 18.8 mm, vias 0 -> 2
- net /SWCLK: track 0.00 -> 18.2 mm
- net /RF_EN: track 5.32 -> 23.3 mm, vias 0 -> 1
- net /WKUP_1: track 10.9 -> 27.9 mm, vias 1 -> 0
- net /RF_TX: track 4.81 -> 21.7 mm, vias 0 -> 1
- net +3V3: track 26.6 -> 37.9 mm, vias 14 -> 20
- net /DATA7: track 5.55 -> 15.3 mm
- net GND: track 62.0 -> 71.6 mm, vias 26 -> 39
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- added copper zone on F.Cu, net +3V3
