File: RF_Remote.kicad_sch (KiCad schematic)
At the start: 92 parts, among them J1 JTAG, J2 UART, J6 CH_USB_C, SW1 NRST, SW2 BOOT, SW3 NRST, SW4 NRST, U1 STM32U031R8Ix, U2 AP7343D-33W5, U3 MICRF112YMU-TR, U4 MCP73833, Y1 25MHz, Y2 32.786KHz, Y3 13.56MHz

Commit message: Routing progress
Parts:
- removed C4, C9: 12p, Capacitor_SMD:C_0603_1608Metric, symbol Device:C_Small
- removed C8: 100n, Capacitor_SMD:C_0603_1608Metric, symbol Device:C_Small
- removed TP2: 5V, TestPoint:TestPoint_Pad_D1.5mm, symbol Connector:TestPoint
- removed U1: STM32U031R8Ix, Package_BGA:UFBGA-64_5x5mm_Layout8x8_P0.5mm, symbol MCU_ST_STM32U0:STM32U031R8Ix
- removed Y1: 25MHz, Crystal:Crystal_SMD_3225-4Pin_3.2x2.5mm, symbol Device:Crystal_GND24_Small
- added TP6: 3v3, TestPoint:TestPoint_Pad_D1.5mm, symbol Connector:TestPoint
- added TP7: GND, TestPoint:TestPoint_Pad_D1.5mm, symbol Connector:TestPoint
- added U5: STM32U031G6Yx, Package_CSP:ST_WLCSP-27_2.34x2.55mm_Layout9x6_P0.4mm_Stagger, symbol MCU_ST_STM32U0:STM32U031G6Yx
- renumbered C12 to C10, C13 to C12, C14 to C13, C15 to C14, C16 to C15, C17 to C16, C18 to C17, C19 to C18, C20 to C19, C21 to C20, C22 to C21, C23 to C22, C24 to C23, C25 to C24, C26 to C25, C27 to C26, C28 to C27, C3 to C4, C6 to C5, C5 to C6, C10 to C9, D11 to D1, D3 to D11, D4 to D12, D5 to D13, D6 to D14, D1 to D2, D12 to D3, D2 to D4, D13 to D5, D14 to D6, J6 to J3, R22 to R10, R5 to R11, R15 to R12, R16 to R13, R6 to R14, R17 to R15, R18 to R16, R7 to R17, R9 to R18, R10 to R19, R11 to R20, R12 to R21, R19 to R3, R3 to R4, R20 to R5, R13 to R6, R14 to R7, R4 to R8, R21 to R9, TP3 to TP1, TP4 to TP2, TP1 to TP3, TP5 to TP4, TP6 to TP5
Connections:
- net +3.3VA: now also U5.F9 (VDDA)
- net +3V3: now also TP6.1, U5.B7 (VDD)
- net BOOT: now also U5.A6 (PF3)
- net DATA0: now also U5.F3 (PB0)
- net DATA1: now also U5.F1 (PB1)
- net DATA2: now also U5.B3 (PB5)
- net DATA3: now also U5.A2 (PB6)
- net DATA4: now also U5.A4 (PB7)
- net DATA5: now also U5.D5 (PA6)
- net DATA6: now also U5.E4 (PA7)
- net DATA7: now also U5.E2 (PA8)
- net GND: now also TP7.1, U5.A8 (VSS)
- net LSE_I: now also U5.B9 (PC14)
- net LSE_O: now also U5.C8 (PC15)
- net NRST: now also U5.D9 (PF2)
- net RF_EN: now also U5.F7 (PA3)
- net RF_TX: now also U5.E8 (PA2)
- net STATUS: now also U5.E6 (PA5)
- net WKUP_1: now also U5.C6 (PA0)
- net WKUP_2: now also U5.D7 (PA1)
- net at J2.2 (Pin_2), TP2.1: now also U5.D1 (PA10)
- net at J2.3 (Pin_3), TP1.1: now also U5.D3 (PA9)
- net at R6.2, R7.1: now also U5.F5 (PA4)
- net SWO: no longer names the net of J1.6 (SWO)
- no-connect marks 35 -> 10
Other:
- note removed: "TODO: no bga"
- moved on the sheet: C10, C13, C2, C4, C6, C7, D1, D10, D3, D5, D6, D7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

Commit message: Layout progress
Parts:
- removed C4, C6, C7: 100n, Capacitor_SMD:C_0603_1608Metric, symbol Device:C_Small
- removed TP4: 3v3, TestPoint:TestPoint_Pad_D1.5mm, symbol Connector:TestPoint
- removed TP5: GND, TestPoint:TestPoint_Pad_D1.5mm, symbol Connector:TestPoint
- added JP2: SENS, Jumper:SolderJumper-2_P1.3mm_Open_TrianglePad1.0x1.5mm, symbol Jumper:SolderJumper_2_Open
- renumbered C15 to C10, C16 to C11, C17 to C12, C18 to C13, C19 to C14, C20 to C15, C21 to C16, C22 to C17, C23 to C18, C24 to C19, C5 to C2, C25 to C20, C26 to C21, C27 to C22, C10 to C3, C2 to C4, C9 to C5, C11 to C6, C13 to C7, C12 to C8, C14 to C9, D4 to D10, D3 to D2, D5 to D3, D6 to D4, D7 to D5, D8 to D6, D9 to D7, D10 to D8, D2 to D9, JP2 to JP3, R3 to R1, R2 to R10, R4 to R11, R8 to R12, R6 to R13, R7 to R14, R11 to R15, R14 to R16, R5 to R2, R9 to R3, R10 to R4, R12 to R5, R13 to R6, R15 to R7, R1 to R8, R16 to R9, TP3 to TP1, TP1 to TP2, TP2 to TP3, TP6 to TP4, TP7 to TP5, U5 to U1, Y2 to Y1, Y3 to Y2
Connections:
- net +BATT: now also JP2.2 (B); no longer R13.1
- new net: JP2.1 (A), R13.1
Other:
- moved on the sheet: C4, TP2, TP3

Commit message: Layout v1
Parts:
- removed TP1, TP2: TX, TestPoint:TestPoint_Pad_D1.5mm, symbol Connector:TestPoint
- removed TP3: RX, TestPoint:TestPoint_Pad_D1.5mm, symbol Connector:TestPoint
- AE1: footprint (none) -> TestPoint:TestPoint_THTPad_D1.0mm_Drill0.5mm
- renumbered TP4 to TP2, TP5 to TP3

Commit message: Cleaned up layout
Parts:
- removed J2: UART, Connector_PinHeader_2.54mm:PinHeader_1x04_P2.54mm_Vertical, symbol Connector:Conn_01x04_Pin
- removed U1: STM32U031G6Yx, Package_CSP:ST_WLCSP-27_2.34x2.55mm_Layout9x6_P0.4mm_Stagger, symbol MCU_ST_STM32U0:STM32U031G6Yx
- added C5: 100n, Capacitor_SMD:C_0603_1608Metric, symbol Device:C_Small
- added U1: STM32U031K4Ux, Package_DFN_QFN:QFN-32-1EP_5x5mm_P0.5mm_EP3.45x3.45mm, symbol MCU_ST_STM32U0:STM32U031K4Ux
- renumbered C9 to C10, C10 to C11, C11 to C12, C12 to C13, C13 to C14, C14 to C15, C15 to C16, C16 to C17, C17 to C18, C18 to C19, C19 to C20, C20 to C21, C21 to C22, C22 to C23, C4 to C3, C3 to C4, C5 to C6, C6 to C7, C7 to C8, C8 to C9, J3 to J2, TP2 to TP1, TP3 to TP2
Connections:
- net +3.3VA: now also U1.5 (VDDA)
- net +3V3: now also C5.1, U1.1 (VDD), U1.17 (VDD)
- net BOOT: now also U1.31 (PF3)
- net DATA0: now also U1.14 (PB0)
- net DATA1: now also U1.15 (PB1)
- net DATA2: now also U1.27 (PB4)
- net DATA3: now also U1.28 (PB5)
- net DATA4: now also U1.29 (PB6)
- net DATA5: now also U1.12 (PA6)
- net DATA6: now also U1.13 (PA7)
- net DATA7: now also U1.18 (PA8)
- net GND: now also C5.2, U1.16 (VSS), U1.32 (VSS), U1.33 (VSS)
- net LSE_I: now also U1.2 (PC14)
- net LSE_O: now also U1.3 (PC15)
- net NRST: now also U1.4 (PF2)
- net RF_EN: now also U1.9 (PA3)
- net RF_TX: now also U1.8 (PA2)
- net STATUS: now also U1.11 (PA5)
- net SWCLK: now also U1.24 (PA14)
- net SWDIO: now also U1.23 (PA13)
- net WKUP_1: now also U1.6 (PA0)
- net WKUP_2: now also U1.7 (PA1)
- net at R13.2, R14.1: now also U1.10 (PA4)
- net SWO: now reaches J1.6 (SWO)
- net SWO: now also U1.26 (PB3)
- no-connect marks 10 -> 13
Other:
- moved on the sheet: C3, JP2, R13, R14
